Commit message: Add husky prefix to all the link names in this package

File: husky_description/urdf/accessories/kinect_camera.urdf.xacro (robot description, xacro)
@@ -29,5 +29,5 @@
     <!-- Create kinect reference frame -->
     <!-- Add mesh for kinect -->
-    <link name="${prefix}_link">
+    <link name="$(arg robot_namespace)/${prefix}_link">
       <origin xyz="0 0 0" rpy="0 0 0"/>
       <visual>
@@ -45,8 +45,8 @@
     <joint name="${prefix}_optical_joint" type="fixed">
       <origin xyz="0 0 0" rpy="-1.5708 0 -1.5708"/>
-      <parent link="${prefix}_link"/>
-      <child link="${prefix}_frame_optical"/>
+      <parent link="$(arg robot_namespace)/${prefix}_link"/>
+      <child link="$(arg robot_namespace)/${prefix}_frame_optical"/>
     </joint>
-    <link name="${prefix}_frame_optical"/>
+    <link name="$(arg robot_namespace)/${prefix}_frame_optical"/>
     <gazebo reference="${prefix}_link">
       <sensor type="depth" name="${prefix}">

File: husky_description/urdf/accessories/sensor_arch.urdf.xacro (robot description, xacro)
@@ -3,5 +3,5 @@
     <xacro:macro name="sensor_arch" params="prefix parent size:=510 *origin">
         <!-- Spawn the sensor arch link -->
-        <link name="${prefix}sensor_arch_mount_link">
+        <link name="$(arg robot_namespace)/${prefix}sensor_arch_mount_link">
              <origin xyz="0 0 0" rpy="0 0 0"/>
              <visual>
@@ -20,6 +20,6 @@
         <joint name="${prefix}sensor_arch_mount" type="fixed">
              <xacro:insert_block name="origin"/>
-             <parent link="${parent}"/>
-             <child link="${prefix}sensor_arch_mount_link"/>
+             <parent link="$(arg robot_namespace)/${parent}"/>
+             <child link="$(arg robot_namespace)/${prefix}sensor_arch_mount_link"/>
         </joint>
     </xacro:macro>

File: husky_description/urdf/accessories/sick_lms1xx_mount.urdf.xacro (robot description, xacro)
@@ -28,5 +28,5 @@
   <xacro:include filename="$(find lms1xx)/urdf/sick_lms1xx.urdf.xacro" />
   <xacro:macro name="sick_lms1xx_mount" params="prefix">
-    <link name="${prefix}_laser_mount">
+    <link name="$(arg robot_namespace)/${prefix}_laser_mount">
       <visual>
         <origin xyz="0 0 0" rpy="0 0 ${-M_PI/2}" />
@@ -46,6 +46,6 @@
       <!-- This offset is from the base of the bracket to the LIDAR's focal point. -->
       <origin xyz="0.0352 0 0.0566" rpy="${M_PI} 0 0" />
-      <parent link="${prefix}_laser_mount" />
-      <child link="${prefix}_laser" />
+      <parent link="$(arg robot_namespace)/${prefix}_laser_mount" />
+      <child link="$(arg robot_namespace)/${prefix}_laser" />
     </joint>
   </xacro:macro>

File: husky_description/urdf/decorations.urdf.xacro (robot description, xacro)
@@ -26,5 +26,5 @@
     <xacro:property name="husky_rear_bumper_extend" value="$(optenv HUSKY_REAR_BUMPER_EXTEND 0)" />
     <!-- Spawn Husky chassis -->
-    <link name="top_chassis_link">
+    <link name="$(arg robot_namespace)/top_chassis_link">
       <visual>
         <origin xyz="0 0 0" rpy="0 0 0" />
@@ -36,10 +36,10 @@
     <!-- Attach chassis to the robot -->
     <joint name="top_chassis_joint" type="fixed">
-      <parent link="base_link" />
-      <child link="top_chassis_link" />
+      <parent link="$(arg robot_namespace)/base_link" />
+      <child link="$(arg robot_namespace)/top_chassis_link" />
     </joint>
     <xacro:if value="$(optenv HUSKY_USER_RAIL_ENABLED true)">
       <!-- Spawn user rails -->
-      <link name="user_rail_link">
+      <link name="$(arg robot_namespace)/user_rail_link">
         <visual>
           <geometry>
@@ -51,10 +51,10 @@
       <joint name="user_rail" type="fixed">
         <origin xyz="0.272 0 0.245" rpy="0 0 0" />
-        <parent link="base_link" />
-        <child link="user_rail_link" />
+        <parent link="$(arg robot_namespace)/base_link" />
+        <child link="$(arg robot_namespace)/user_rail_link" />
       </joint>
     </xacro:if>
     <!-- Spawn front bumper link -->
-    <link name="front_bumper_link">
+    <link name="$(arg robot_namespace)/front_bumper_link">
       <visual>
         <geometry>
@@ -66,9 +66,9 @@
     <joint name="front_bumper" type="fixed">
       <origin xyz="${0.48 + husky_front_bumper_extend} 0 0.091" rpy="0 0 0" />
-      <parent link="base_link" />
-      <child link="front_bumper_link" />
+      <parent link="$(arg robot_namespace)/base_link" />
+      <child link="$(arg robot_namespace)/front_bumper_link" />
     </joint>
     <xacro:if value="${husky_front_bumper_extend}">
-      <link name="front_bumper_extension_link">
+      <link name="$(arg robot_namespace)/front_bumper_extension_link">
           <visual>
               <geometry>
@@ -79,10 +79,10 @@
       <joint name="front_bumper_extension" type="fixed">
         <origin xyz="${0.48 + husky_front_bumper_extend} 0 0.091" rpy="0 0 0" />
-        <parent link="base_link" />
-        <child link="front_bumper_extension_link" />
+        <parent link="$(arg robot_namespace)/base_link" />
+        <child link="$(arg robot_namespace)/front_bumper_extension_link" />
       </joint>
     </xacro:if>
     <!-- Spawn rear bumper link -->
-    <link name="rear_bumper_link">
+    <link name="$(arg robot_namespace)/rear_bumper_link">
       <visual>
         <geometry>
@@ -94,9 +94,9 @@
     <joint name="rear_bumper" type="fixed">
       <origin xyz="${-0.48 - husky_rear_bumper_extend} 0 0.091" rpy="0 0 ${M_PI}" />
-      <parent link="base_link" />
-      <child link="rear_bumper_link" />
+      <parent link="$(arg robot_namespace)/base_link" />
+      <child link="$(arg robot_namespace)/rear_bumper_link" />
     </joint>
     <xacro:if value="${husky_rear_bumper_extend}">
-      <link name="rear_bumper_extension_link">
+      <link name="$(arg robot_namespace)/rear_bumper_extension_link">
           <visual>
               <geometry>
@@ -107,6 +107,6 @@
       <joint name="rear_bumper_extension" type="fixed">
         <origin xyz="${-0.48 - husky_rear_bumper_extend} 0 0.091" rpy="0 0 ${M_PI}" />
-        <parent link="base_link" />
-        <child link="rear_bumper_extension_link" />
+        <parent link="$(arg robot_namespace)/base_link" />
+        <child link="$(arg robot_namespace)/rear_bumper_extension_link" />
       </joint>
     </xacro:if>
@@ -114,5 +114,5 @@
       <!-- Spawn the top plate -->
       <xacro:if value="$(optenv HUSKY_LARGE_TOP_PLATE false)">
-        <link name="top_plate_link">
+        <link name="$(arg robot_namespace)/top_plate_link">
           <visual>
             <origin xyz="0 0 0" rpy="0 0 0" />
@@ -130,23 +130,23 @@
         <!-- Attach top plate -->
         <joint name="top_plate_joint" type="fixed">
-          <parent link="base_link" />
-          <child link="top_plate_link"/>
+          <parent link="$(arg robot_namespace)/base_link" />
+          <child link="$(arg robot_namespace)/top_plate_link"/>
           <origin xyz="0.0812 0 0.225" rpy="0 0 0"/>
         </joint>
         <!-- Top plate front link -->
         <joint name="top_plate_front_joint" type="fixed">
-          <parent link="top_plate_link" />
-          <child link="top_plate_front_link"/>
+          <parent link="$(arg robot_namespace)/top_plate_link" />
+          <child link="$(arg robot_namespace)/top_plate_front_link"/>
           <origin xyz="0.4125 0 0.00672" rpy="0 0 0"/>
         </joint>
         <!-- Top plate rear link-->
         <joint name="top_plate_rear_joint" type="fixed">
-          <parent link="top_plate_link" />
-          <child link="top_plate_rear_link"/>
+          <parent link="$(arg robot_namespace)/top_plate_link" />
+          <child link="$(arg robot_namespace)/top_plate_rear_link"/>
           <origin xyz="-0.4125 0 0.00672" rpy="0 0 0"/>
         </joint>
       </xacro:if>
       <xacro:unless value="$(optenv HUSKY_LARGE_TOP_PLATE false)">
-        <link name="top_plate_link">
+        <link name="$(arg robot_namespace)/top_plate_link">
           <visual>
             <origin xyz="0 0 0" rpy="0 0 0" />
@@ -164,23 +164,23 @@
         <!-- Attach top plate -->
         <joint name="top_plate_joint" type="fixed">
-          <parent link="base_link" />
-          <child link="top_plate_link"/>
+          <parent link="$(arg robot_namespace)/base_link" />
+          <child link="$(arg robot_namespace)/top_plate_link"/>
           <origin xyz="0.0812 0 0.245" rpy="0 0 0"/>
         </joint>
         <!-- Top plate front link -->
         <joint name="top_plate_front_joint" type="fixed">
-          <parent link="top_plate_link" />
-          <child link="top_plate_front_link"/>
+          <parent link="$(arg robot_namespace)/top_plate_link" />
+          <child link="$(arg robot_namespace)/top_plate_front_link"/>
           <origin xyz="0.36367 0 0.00639" rpy="0 0 0"/>
         </joint>
         <!-- Top plate rear link-->
         <joint name="top_plate_rear_joint" type="fixed">
-          <parent link="top_plate_link" />
-          <child link="top_plate_rear_link"/>
+          <parent link="$(arg robot_namespace)/top_plate_link" />
+          <child link="$(arg robot_namespace)/top_plate_rear_link"/>
           <origin xyz="-0.36633 0 0.00639" rpy="0 0 0"/>
         </joint>
       </xacro:unless>
-      <link name="top_plate_front_link"/>
-      <link name="top_plate_rear_link"/>
+      <link name="$(arg robot_namespace)/top_plate_front_link"/>
+      <link name="$(arg robot_namespace)/top_plate_rear_link"/>
     </xacro:if>
   </xacro:macro>

File: husky_description/urdf/husky.urdf.xacro (robot description, xacro)
@@ -52,5 +52,5 @@
   <xacro:property name="wheel_radius" value="0.1651" />
   <!-- Base link is the center of the robot's bottom plate -->
-  <link name="base_link">
+  <link name="$(arg robot_namespace)/base_link">
     <visual>
       <origin xyz="0 0 0" rpy="0 0 0" />
@@ -73,12 +73,12 @@
   </link>
   <!-- Base footprint is on the ground under the robot -->
-  <link name="base_footprint"/>
+  <link name="$(arg robot_namespace)/base_footprint"/>
   <joint name="base_footprint_joint" type="fixed">
     <origin xyz="0 0 ${wheel_vertical_offset - wheel_radius}" rpy="0 0 0" />
-    <parent link="base_link" />
-    <child link="base_footprint" />
+    <parent link="$(arg robot_namespace)/base_link" />
+    <child link="$(arg robot_namespace)/base_footprint" />
   </joint>
   <!-- Interial link stores the robot's inertial information -->
-  <link name="inertial_link">
+  <link name="$(arg robot_namespace)/inertial_link">
     <inertial>
       <mass value="46.034" />
@@ -89,14 +89,14 @@
   <joint name="inertial_joint" type="fixed">
     <origin xyz="0 0 0" rpy="0 0 0" />
-    <parent link="base_link" />
-    <child link="inertial_link" />
+    <parent link="$(arg robot_namespace)/base_link" />
+    <child link="$(arg robot_namespace)/inertial_link" />
   </joint>
   <!-- IMU Link is the standard mounting position for the UM6 IMU.-->
   <!-- Can be modified with environment variables in /etc/ros/setup.bash -->
-  <link name="imu_link"/>
+  <link name="$(arg robot_namespace)/imu_link"/>
   <joint name="imu_joint" type="fixed">
     <origin xyz="$(optenv HUSKY_IMU_XYZ 0.19 0 0.149)" rpy="$(optenv HUSKY_IMU_RPY 0 -1.5708 3.1416)" />
-    <parent link="base_link" />
-    <child link="imu_link" />
+    <parent link="$(arg robot_namespace)/base_link" />
+    <child link="$(arg robot_namespace)/imu_link" />
   </joint>
   <gazebo reference="imu_link">
@@ -105,8 +105,8 @@
   <joint name="target_joint" type="fixed">
     <origin xyz="0 0 0.255" rpy="0 0 0" />
-    <parent link="base_link" />
-    <child link="target_link" />
+    <parent link="$(arg robot_namespace)/base_link" />
+    <child link="$(arg robot_namespace)/target_link" />
   </joint>
-  <link name="target_link">
+  <link name="$(arg robot_namespace)/target_link">
     <inertial>
       <origin xyz="0 0 0"/>
@@ -146,6 +146,6 @@
     <joint name="laser_mount_joint" type="fixed">
       <origin xyz="$(arg laser_xyz)" rpy="$(arg laser_rpy)" />
-      <parent link="top_plate_link" />
-      <child link="base_laser_mount" />
+      <parent link="$(arg robot_namespace)/top_plate_link" />
+      <child link="$(arg robot_namespace)/base_laser_mount" />
     </joint>
   </xacro:if>
@@ -156,6 +156,6 @@
     <joint name="kinect_frame_joint" type="fixed">
       <origin xyz="$(arg kinect_xyz)" rpy="$(arg kinect_rpy)" />
-      <parent link="sensor_arch_mount_link"/>
-      <child link="camera_link"/>
+      <parent link="$(arg robot_namespace)/sensor_arch_mount_link"/>
+      <child link="$(arg robot_namespace)/camera_link"/>
     </joint>
     <xacro:kinect_camera prefix="camera" robot_namespace="$(arg robot_namespace)"/>
@@ -171,5 +171,5 @@
       <robotNamespace>$(arg robot_namespace)</robotNamespace>
       <updateRate>50.0</updateRate>
-      <bodyName>base_link</bodyName>
+      <bodyName>$(arg robot_namespace)/base_link</bodyName>
       <topicName>imu/data</topicName>
       <accelDrift>0.005 0.005 0.005</accelDrift>
@@ -185,6 +185,6 @@
       <robotNamespace>$(arg robot_namespace)</robotNamespace>
       <updateRate>40</updateRate>
-      <bodyName>base_link</bodyName>
-      <frameId>base_link</frameId>
+      <bodyName>$(arg robot_namespace)/base_link</bodyName>
+      <frameId>$(arg robot_namespace)/base_link</frameId>
       <topicName>navsat/fix</topicName>
       <velocityTopicName>navsat/vel</velocityTopicName>

File: husky_description/urdf/wheel.urdf.xacro (robot description, xacro)
@@ -23,5 +23,5 @@
 <robot xmlns:xacro="http://ros.org/wiki/xacro" name="husky_wheel">
 	<xacro:macro name="husky_wheel" params="wheel_prefix *joint_pose">
-		<link name="${wheel_prefix}_wheel_link">
+		<link name="$(arg robot_namespace)/${wheel_prefix}_wheel_link">
 			<inertial>
 				<mass value="2.637" />
@@ -50,6 +50,6 @@
 		</gazebo>
 		<joint name="${wheel_prefix}_wheel" type="continuous">
-			<parent link="base_link"/>
-			<child link="${wheel_prefix}_wheel_link"/>
+			<parent link="$(arg robot_namespace)/base_link"/>
+			<child link="$(arg robot_namespace)/${wheel_prefix}_wheel_link"/>
 			<xacro:insert_block name="joint_pose"/>
 			<axis xyz="0 1 0" rpy="0 0 0" />
