Commit message: Initial commit for putting a target on the husky and removing limits on angular/linear velocity and acceleration

File: husky_description/urdf/husky.urdf.xacro (robot description, xacro)
@@ -101,4 +101,38 @@
   <gazebo reference="imu_link">
   </gazebo>
+  <!-- Target link is where the Apriltag is -->
+  <joint name="target_joint" type="fixed">
+    <origin xyz="0 0 0.255" rpy="0 0 0" />
+    <parent link="base_link" />
+    <child link="target_link" />
+  </joint>
+  <link name="target_link">
+    <inertial>
+      <origin xyz="0 0 0"/>
+      <mass value="1.0"/>
+      <inertia ixx="1.0" ixy="0.0" ixz="0.0" iyy="1.0" iyz="0.0" izz="1.0"/>
+    </inertial>
+    <collision>
+      <origin xyz="0 0 0" rpy="0 0 0" />
+      <geometry>
+        <box size="0.8 0.8 0.001" />
+      </geometry>
+    </collision>
+    <visual>
+      <origin xyz="0 0 0" rpy="0 0 0" />
+      <geometry>
+        <!--mesh filename="package://rotors_description/meshes/target.dae" scale="1 1 1" /-->
+        <mesh filename="$(find rotors_description)/meshes/target.dae" scale="1 1 1" />
+      </geometry>
+    </visual>
+  </link>
+  <xacro:include filename="$(find rotors_description)/urdf/component_snippets.xacro" />
+  <xacro:default_imu namespace="target" parent_link="target_link" />
+  <!-- <gazebo>
+    <plugin name="landing_target_plugin" filename="librotors_gazebo_landing_target_plugin.so">
+      <robotNamespace>husky</robotNamespace>
+      <linkName>husky/target_joint</linkName>
+    </plugin>
+  </gazebo> -->
   <!-- Husky wheel macros -->
   <xacro:husky_wheel wheel_prefix="front_left">
@@ -135,4 +169,5 @@
     <xacro:kinect_camera prefix="camera" robot_namespace="$(arg robot_namespace)"/>
   </xacro:if>
+  <rosparam command="load" file="$(find husky_description)/urdf/gazebo_ros_control.yaml" />
   <gazebo>
     <plugin name="gazebo_ros_control" filename="libgazebo_ros_control.so">

Commit message: Fixed target tracking

File: husky_description/urdf/husky.urdf.xacro (robot description, xacro)
@@ -123,15 +123,8 @@
       <origin xyz="0 0 0" rpy="0 0 0" />
       <geometry>
-        <!--mesh filename="package://rotors_description/meshes/target.dae" scale="1 1 1" /-->
-        <mesh filename="$(find rotors_description)/meshes/target.dae" scale="1 1 1" />
+        <mesh filename="$(find husky_description)/meshes/target.dae" scale="1 1 1"/>
       </geometry>
     </visual>
   </link>
-  <!-- <gazebo>
-    <plugin name="husky_plugin" filename="librotors_gazebo_husky_plugin.so">
-      <robotNamespace>husky</robotNamespace>
-      <linkName>base_link</linkName>
-    </plugin>
-  </gazebo> -->
   <!-- Husky wheel macros -->
   <xacro:husky_wheel wheel_prefix="front_left">

Commit message: TRAILab-specific changes to husky repo

File: husky_description/urdf/husky.urdf.xacro (robot description, xacro)
@@ -22,21 +22,11 @@
 -->
 <robot name="husky" xmlns:xacro="http://ros.org/wiki/xacro">
-  <xacro:arg name="laser_enabled" default="false" />
-  <xacro:arg name="laser_xyz" default="$(optenv HUSKY_LMS1XX_XYZ 0.2206 0.0 0.00635)" />
-  <xacro:arg name="laser_rpy" default="$(optenv HUSKY_LMS1XX_RPY 0.0 0.0 0.0)" />
-  <xacro:arg name="realsense_enabled" default="false" />
-  <xacro:arg name="realsense_xyz" default="$(optenv HUSKY_REALSENSE_XYZ 0 0 0)" />
-  <xacro:arg name="realsense_rpy" default="$(optenv HUSKY_REALSENSE_RPY 0 0 0)" />
-  <xacro:arg name="realsense_mount" default="$(optenv HUSKY_REALSENSE_MOUNT_FRAME sensor_arch_mount_link)" />
   <xacro:property name="husky_front_bumper_extend" value="$(optenv HUSKY_FRONT_BUMPER_EXTEND 0)" />
   <xacro:property name="husky_rear_bumper_extend" value="$(optenv HUSKY_REAR_BUMPER_EXTEND 0)" />
   <xacro:arg name="robot_namespace" default="/" />
-  <xacro:arg name="urdf_extras" default="empty.urdf" />
+  <xacro:arg name="urdf_extras" default="$(find husky_description)/urdf/extras.urdf.xacro" />
   <!-- Included URDF/XACRO Files -->
   <xacro:include filename="$(find husky_description)/urdf/decorations.urdf.xacro" />
   <xacro:include filename="$(find husky_description)/urdf/wheel.urdf.xacro" />
-  <xacro:include filename="$(find husky_description)/urdf/accessories/intel_realsense.urdf.xacro"/>
-  <xacro:include filename="$(find husky_description)/urdf/accessories/sick_lms1xx_mount.urdf.xacro"/>
-  <xacro:include filename="$(find husky_description)/urdf/accessories/sensor_arch.urdf.xacro"/>
   <xacro:property name="M_PI" value="3.14159"/>
   <!-- Base Size -->
@@ -116,39 +106,6 @@
   </xacro:husky_wheel>
   <xacro:husky_decorate />
-  <xacro:if value="$(arg laser_enabled)">
-    <xacro:sick_lms1xx_mount prefix="base"/>
-    <xacro:sick_lms1xx frame="base_laser" topic="scan" robot_namespace="$(arg robot_namespace)"/>
-    <joint name="laser_mount_joint" type="fixed">
-      <origin xyz="$(arg laser_xyz)" rpy="$(arg laser_rpy)" />
-      <parent link="top_plate_link" />
-      <child link="base_laser_mount" />
-    </joint>
-  </xacro:if>
-  <!--
-    top sensor arch; include this if we have realsense enabled
-    keep this as a property to make it easier to add multiple conditions, should we need
-    the top bar for any additional sensors in the future
-  -->
-  <xacro:property name="topbar_needed_realsense" value="$(arg realsense_enabled)" />
-  <xacro:if value="${topbar_needed_realsense}">
-    <xacro:sensor_arch prefix="" parent="top_plate_link">
-      <origin xyz="-0.35 0 0.51" rpy="0 0 -3.14"/>
-    </xacro:sensor_arch>
-  </xacro:if>
-  <!-- add the intel realsense to the topbar if needed -->
-  <xacro:if value="$(arg realsense_enabled)">
-    <link name="realsense_mountpoint"/>
-    <joint name="realsense_mountpoint_joint" type="fixed">
-      <origin xyz="0 0 0" rpy="0 0 -3.14159" />
-      <parent link="$(arg realsense_mount)"/>
-      <child link="realsense_mountpoint" />
-    </joint>
-    <xacro:intel_realsense_mount prefix="camera" topic="realsense" parent_link="realsense_mountpoint"/>
-  </xacro:if>
   <gazebo>
-    <plugin name="gazebo_ros_control" filename="libgazebo_ros_control.so">
-      <robotNamespace>$(arg robot_namespace)</robotNamespace>
-      <legacyModeNS>true</legacyModeNS>
-    </plugin>
+    <plugin name="gazebo_ros_control" filename="libgazebo_ros_control.so" />
   </gazebo>
   <gazebo>
@@ -183,3 +140,4 @@
   <!-- Optional custom includes. -->
   <xacro:include filename="$(arg urdf_extras)" />
+  <xacro:apriltag parent_link="base_link" />
 </robot>
